File: pcb-joycon.kicad_pcb (KiCad board)
At the start: 2 copper layers, 189.2 x 120.6 mm, 57 parts, among them U1 Arduino_Pro_Micro, U2 TRRS

Commit message: minor edit
Routing:
- net VCC: track 62.4 -> 61.8 mm
Changed lines of the file:
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@@
   (segment (start 66.02 31.73) (end 71.12 36.83) (width 0.35) (layer "B.Cu") (net 44))
   (segment (start 71.12 36.83) (end 78.105 36.83) (width 0.35) (layer "B.Cu") (net 44))
-  (segment (start 95.885 19.685) (end 99.06 22.86) (width 0.35) (layer "F.Cu") (net 48))
-  (segment (start 99.06 22.86) (end 99.06 26.035) (width 0.35) (layer "F.Cu") (net 48))
-  (segment (start 76.2 19.685) (end 76.835 20.32) (width 0.35) (layer "F.Cu") (net 48))
+  (segment (start 76.2 19.685) (end 95.885 19.685) (width 0.35) (layer "F.Cu") (net 48))
   (segment (start 70.0125 19.685) (end 64.21625 19.685) (width 0.35) (layer "F.Cu") (net 48))
-  (segment (start 77.47 19.685) (end 95.885 19.685) (width 0.35) (layer "F.Cu") (net 48))
   (segment (start 63.02 20.88125) (end 63.02 24.37) (width 0.35) (layer "F.Cu") (net 48))
   (segment (start 72.5525 21.59) (end 72.5525 21.615) (width 0.35) (layer "F.Cu") (net 48))
@@
   (segment (start 64.21625 19.685) (end 63.02 20.88125) (width 0.35) (layer "F.Cu") (net 48))
   (segment (start 74.27 21.615) (end 72.5525 21.615) (width 0.18) (layer "F.Cu") (net 48))
-  (segment (start 76.835 20.32) (end 77.47 19.685) (width 0.35) (layer "F.Cu") (net 48))
+  (segment (start 99.06 22.86) (end 99.06 26.035) (width 0.35) (layer "F.Cu") (net 48))
   (segment (start 76.2 19.685) (end 70.0125 19.685) (width 0.35) (layer "F.Cu") (net 48))
+  (segment (start 95.885 19.685) (end 99.06 22.86) (width 0.35) (layer "F.Cu") (net 48))
   (segment (start 99.06 26.035) (end 93.345 31.75) (width 0.35) (layer "F.Cu") (net 48))
   (segment (start 70.0125 19.685) (end 68.1125 21.585) (width 0.25) (layer "F.Cu") (net 48))
